File: mt3608.kicad_sch (KiCad schematic)
At the start: 10 parts, among them U1 MT3608

Commit message: Added an example schematic for the OLED devices
Parts:
- renumbered C1 to C13, C2 to C14, C3 to C15, C4 to C16, D1 to D3, R1 to R10, R2 to R11, R3 to R12, U1 to U3
